Commit message: feat: implement pybullet simulation scene

File: assets/ur5/ur5_joint_limited_robot.urdf (robot description, URDF)
Before this commit: robot ur5, 11 links, 10 joints
Links:
- added link suction_cup_link, mass 0.05; collision cylinder length=0.012 radius=0.014; collision cylinder length=0.025 radius=0.007
Joints:
- added joint wrist_3_link-suction_cup_fixed_joint: type fixed, parent wrist_3_link, child suction_cup_link, origin xyz=0 0.0823 0 rpy=-1.57079632679 0 0
